Commit message: add chassis_urdf

File: src/gluon/urdf/gluon.urdf (robot description, URDF)
Before this commit: robot gluon, 9 links, 8 joints
Links:
- removed link center_link
Joints:
- removed joint dummy_center_joint
- removed joint left_base_joint
- added joint dummy_joint: type fixed, parent dummy, child base_link, origin xyz=0 0 0 rpy=0 0 0
