Commit message: xacro change

File: src/chasis_urdf/urdf/chasis_urdf.xacro (robot description, xacro)
@@ -3,5 +3,7 @@
      Commit Version: 1.6.0-4-g7f85cfe  Build Version: 1.6.7995.38578
      For more information, please see http://wiki.ros.org/sw_urdf_exporter -->
-<xacro:macro name="joint_trans" params="joint_name">
+<robot
+  name="chasis_urdf" xmlns:xacro="http://wiki.ros.org/xacro">
+  <xacro:macro name="joint_trans" params="joint_name">
         <!-- Transmission is important to link the joints and the controller -->
         <transmission name="${joint_name}_trans">
@@ -16,6 +18,4 @@
         </transmission>
     </xacro:macro>
-<robot
-  name="chasis_urdf" xmlns:xacro="http://wiki.ros.org/xacro">
   <link name="base_link">
     <inertial>
@@ -285,8 +285,8 @@
             <odometryTopic>odom</odometryTopic>
             <odometryFrame>odom</odometryFrame>
-            <leftFrontJoint>front_left</leftFrontJoint>
-            <rightFrontJoint>front_right</rightFrontJoint>
-            <leftRearJoint>back_left</leftRearJoint>
-            <rightRearJoint>back_right</rightRearJoint>
+            <leftFrontJoint>back_left</leftFrontJoint>
+            <rightFrontJoint>front_left</rightFrontJoint>
+            <leftRearJoint>back_right</leftRearJoint>
+            <rightRearJoint>front_right</rightRearJoint>
             <odometryRate>100</odometryRate>
             <robotBaseFrame>base_footprint</robotBaseFrame>
