Commit message: add_2l46l3_arm

File: src/gluon_2L4_6L3/urdf/dual_arm.urdf (robot description, URDF)
Before this commit: robot dual_arm, 16 links, 15 joints
Links:
- removed link right_1_Link
- removed link right_2_Link
- removed link right_3_Link
- removed link right_4_Link
- removed link right_5_Link
- removed link right_6_Link
- removed link right_base_link
Joints:
- removed joint right_axis_joint_1
- removed joint right_axis_joint_2
- removed joint right_axis_joint_3
- removed joint right_axis_joint_4
- removed joint right_axis_joint_5
- removed joint right_axis_joint_6
- removed joint right_base_joint
- joint left_base_joint: origin xyz=-0.15 0 0.095 rpy=-1.570795 0 1.570795 -> xyz=0.0 0.15 0.095 rpy=0 0 0

File: src/gluon_2L4_6L3/urdf/xtou_dual_arm.urdf (robot description, URDF)
Before this commit: robot dual_arm, 16 links, 15 joints
Links:
- removed link base_link
- removed link right_1_Link
- removed link right_2_Link
- removed link right_3_Link
- removed link right_4_Link
- removed link right_5_Link
- removed link right_6_Link
- removed link right_base_link
- added link center_link, mass 1.088; collision mesh filename=package://gluon/meshes/center_link.STL; visual mesh filename=package://gluon/meshes/center_link.STL
Joints:
- removed joint right_axis_joint_1
- removed joint right_axis_joint_2
- removed joint right_axis_joint_3
- removed joint right_axis_joint_4
- removed joint right_axis_joint_5
- removed joint right_axis_joint_6
- removed joint right_base_joint
- joint dummy_center_joint: child base_link -> center_link
- joint left_base_joint: origin xyz=-0.15 0 0.095 rpy=-1.570795 0 1.570795 -> xyz=0.0 0.15 0.095 rpy=0 0 0; parent base_link -> center_link
